File: can.kicad_sch (KiCad schematic)
At the start: 7 parts, among them J400 Conn_01x03, U400 TJA1042T-3

Commit message: fix: Silkscreen overlaps
Parts:
- C400, C401: footprint Capacitor_SMD:C_0402_1005Metric -> Library:C_0402_1005Metric
- R400: footprint Resistor_SMD:R_0402_1005Metric -> Library:R_0402_1005Metric
Changed lines of the file:
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@@
 			)
 		)
-		(property "Footprint" "Capacitor_SMD:C_0402_1005Metric"
+		(property "Footprint" "Library:C_0402_1005Metric"
 			(at 44.1452 45.72 0)
 			(effects
@@
 			)
 		)
-		(property "Footprint" "Capacitor_SMD:C_0402_1005Metric"
+		(property "Footprint" "Library:C_0402_1005Metric"
 			(at 23.8252 80.01 0)
 			(effects
@@
 			)
 		)
-		(property "Footprint" "Resistor_SMD:R_0402_1005Metric"
+		(property "Footprint" "Library:R_0402_1005Metric"
 			(at 87.884 47.244 90)
 			(effects
