File: microcontroller.kicad_sch (KiCad schematic)
At the start: 52 parts, among them J100 Conn_01x05_Pin, J101 Screw_Terminal_01x02, J102 USB_C_Receptacle_USB2.0_16P, Q100 Si2371EDS, SW100 SKRPANE010, U100 STM32H563RITx, U101 AP2112K-3.3, U102 USBLC6-2SC6, Y100 16MHz

Commit message: fix: Silkscreen overlaps
Parts:
- C101, C102, C104, C105, C107, C109, C110, C111, C112, C113, C117, C118, C119: footprint Capacitor_SMD:C_0402_1005Metric -> Library:C_0402_1005Metric
- R100, R101, R102, R103, R104, R105, R106, R107: footprint Resistor_SMD:R_0402_1005Metric -> Library:R_0402_1005Metric
